File: RoyBoard.kicad_sch (KiCad schematic)
At the start: 336 parts, among them J1 USB_C_Receptacle_USB2.0_16P, SW1 SW_Push, SW10 SW_Push, SW11 SW_Push, SW12 SW_Push, SW13 SW_Push, SW14 SW_Push, SW15 SW_Push, SW16 SW_Push, SW17 SW_Push, SW18 SW_Push, SW19 SW_Push, SW2 SW_Push, SW20 SW_Push, SW21 SW_Push, SW22 SW_Push, SW23 SW_Push, SW24 SW_Push, SW25 SW_Push, SW26 SW_Push, SW27 SW_Push, SW28 SW_Push, SW29 SW_Push, SW3 SW_Push, SW30 SW_Push, SW31 SW_Push, SW32 SW_Push, SW33 SW_Push, SW34 SW_Push, SW35 SW_Push, SW36 SW_Push, SW37 SW_Push, SW38 SW_Push, SW39 SW_Push, SW4 SW_Push, SW40 SW_Push, SW41 SW_Push, SW42 SW_Push, SW43 SW_Push, SW44 SW_Push, SW45 SW_Push, SW46 SW_Push, SW47 SW_Push, SW48 SW_Push, SW49 SW_Push, SW5 SW_Push, SW50 SW_Push, SW51 SW_Push, SW52 SW_Push, SW53 SW_Push, SW54 SW_Push, SW55 SW_Push, SW56 SW_Push, SW57 SW_Push, SW58 SW_Push, SW59 SW_Push, SW6 SW_Push, SW60 SW_Push, SW61 SW_Push, SW62 SW_Push, SW63 SW_Push, SW64 SW_Push, SW65 SW_Push, SW66 SW_Push, SW67 SW_Push, SW68 SW_Push, SW69 SW_Push, SW7 SW_Push, SW70 SW_Push, SW71 SW_Push, SW72 SW_Push, SW73 SW_Push, SW74 SW_Push, SW75 SW_Push, SW76 SW_Push, SW77 SW_Push, SW78 SW_Push, SW79 SW_Push, SW8 SW_Push, SW80 SW_Push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

Commit message: Completed keyboard
Parts:
- removed C1, C10, C11, C12, C13, C14, C15, C16, C17, C18, C19, C2, C20, C21, C22, C23, C24, C25, C26, C27, C28, C29, C3, C30, C31, C32, C33, C34, C35, C36, C37, C38, C39, C4, C40, C41, C42, C43, C44, C45, C46, C47, C48, C49, C5, C50, C51, C52, C53, C54, C55, C56, C57, C58, C59, C6, C60, C61, C62, C63, C64, C65, C66, C67, C68, C69, C7, C70, C71, C72, C73, C74, C75, C76, C77, C78, C79, C8, C80, C81, C82, C9: 1uf, symbol Device:C
- removed D100, D101, D102, D103, D104, D105, D106, D107, D108, D109, D110, D111, D112, D113, D114, D115, D116, D117, D118, D119, D120, D121, D122, D123, D124, D125, D126, D127, D128, D129, D130, D131, D132, D133, D134, D135, D136, D137, D138, D139, D140, D141, D142, D143, D144, D145, D146, D147, D148, D149, D150, D151, D152, D153, D154, D155, D156, D157, D158, D159, D160, D161, D162, D163, D164, D165, D91, D92, D93, D94, D95, D96, D97, D98, D99: SK6812MINI, royboard_footprints:SK6812MINI-E, symbol LED:SK6812MINI
- removed D166: SK6812MINI, LED_SMD:LED_SK6812MINI_PLCC4_3.5x3.5mm_P1.75mm, symbol LED:SK6812MINI
- removed J1: USB_C_Receptacle_USB2.0_16P, symbol Connector:USB_C_Receptacle_USB2.0_16P
- removed R1: 10k, symbol Device:R
- removed U2: CH224K, Package_SO:SSOP-10-1EP_3.9x4.9mm_P1mm_EP2.1x3.3mm, symbol Interface_USB:CH224K
- D85, D86, D87, D88, D89, D90: footprint royboard_footprints:SK6812MINI-E -> royboard_footprints:LED_SK6812MINI_PLCC4_3.5x3.5mm_P1.75mm
- SW54, SW55: footprint PCM_Switch_Keyboard_Cherry_MX:SW_Cherry_MX_PCB_2.25u -> Button_Switch_Keyboard:SW_Cherry_MX_2.25u_PCB
- SW66: footprint PCM_Switch_Keyboard_Cherry_MX:SW_Cherry_MX_PCB_2.75u -> Button_Switch_Keyboard:SW_Cherry_MX_2.75u_PCB
- SW67: footprint PCM_Switch_Keyboard_Cherry_MX:SW_Cherry_MX_PCB_1.25u -> Button_Switch_Keyboard:SW_Cherry_MX_1.25u_PCB
- SW70: footprint PCM_Switch_Keyboard_Cherry_MX:SW_Cherry_MX_PCB_6.25u -> Button_Switch_Keyboard:SW_Cherry_MX_6.25u_PCB
- renumbered SW6 to SW5, SW7 to SW6, SW8 to SW7, SW9 to SW8, SW5 to SW9
Connections:
- no-connect marks 3 -> 1
Other:
- moved on the sheet: U1
