File: PCB/RoyBoard.kicad_pcb (KiCad board)
At the start: 2 copper layers, 369.5 x 136.6 mm, 180 parts, among them SW1 SW_Push, SW10 SW_Push, SW11 SW_Push, SW12 SW_Push, SW13 SW_Push, SW14 SW_Push, SW15 SW_Push, SW16 SW_Push, SW17 SW_Push, SW18 SW_Push, SW19 SW_Push, SW2 SW_Push, SW20 SW_Push, SW21 SW_Push, SW22 SW_Push, SW23 SW_Push, SW24 SW_Push, SW25 SW_Push, SW26 SW_Push, SW27 SW_Push, SW28 SW_Push, SW29 SW_Push, SW3 SW_Push, SW30 SW_Push, SW31 SW_Push, SW32 SW_Push, SW33 SW_Push, SW34 SW_Push, SW35 SW_Push, SW36 SW_Push, SW37 SW_Push, SW38 SW_Push, SW39 SW_Push, SW4 SW_Push, SW40 SW_Push, SW41 SW_Push, SW42 SW_Push, SW43 SW_Push, SW44 SW_Push, SW45 SW_Push, SW46 SW_Push, SW47 SW_Push, SW48 SW_Push, SW49 SW_Push, SW5 SW_Push, SW50 SW_Push, SW51 SW_Push, SW52 SW_Push, SW53 SW_Push, SW54 SW_Push, SW55 SW_Push, SW56 SW_Push, SW57 SW_Push, SW58 SW_Push, SW59 SW_Push, SW6 SW_Push, SW60 SW_Push, SW61 SW_Push, SW62 SW_Push, SW63 SW_Push, SW64 SW_Push, SW65 SW_Push, SW66 SW_Push, SW67 SW_Push, SW68 SW_Push, SW69 SW_Push, SW7 SW_Push, SW70 SW_Push, SW71 SW_Push, SW72 SW_Push, SW73 SW_Push, SW74 SW_Push, SW75 SW_Push, SW76 SW_Push, SW77 SW_Push, SW78 SW_Push, SW79 SW_Push, SW8 SW_Push, SW80 SW_Push, SW81 SW_Push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

Commit message: Added readme and changed silkscreen
Parts:
- removed the G*** at (143.1, 74.3)
- removed the G*** at (74.6, 123.8)
- removed the G*** at (67.0, 53.0)
- removed the G*** at (67.8, 42.8)
- removed the G*** at (337.7, 123.3)
- added G***: LOGO, LOGO, F.Cu at (337.9, 109.4)
- added G***: LOGO, LOGO, B.Cu at (67.9, 47.4)
- added G***: LOGO, LOGO, B.Cu at (339.9, 112.4)
- added G***: LOGO, LOGO, B.Cu at (362.9, 59.4)
Routing:
- net GND: track 994.9 -> 990.7 mm
Other:
- board text added: "Don't, I warned you"
- board text added: "Shibam Roy"
- board text added: "THOCKS!"
- board text added: "This One"
- board text added: "This keyboard is cursed with functionality and coolness, use with caution:)"
- board text removed: "DO NOT SCAN THIS!!"
- board text removed: "RoyBoard made By Shibam Roy"
- board text removed: "What can this be...?"

Commit message: Added CAD models, firmware and 3d renders
Parts:
- SW27: footprint PCM_Switch_Keyboard_Cherry_MX:SW_Cherry_MX_PCB_2.00u -> Button_Switch_Keyboard:SW_Cherry_MX_2.00u_PCB
- moved SW27 0.05 mm to (307.6, 68.8)
Routing:
- net col3: track 568.8 -> 580.9 mm
- net Net-(D27-A): track 16.3 -> 28.3 mm
- net row3: track 329.2 -> 331.8 mm
- net col5: track 622.5 -> 623.2 mm
- net row4: track 372.8 -> 373.4 mm

Commit message: Added new minecraft themed silkscreen
Parts:
- removed the G*** at (337.9, 109.4)
- removed the G*** at (339.9, 112.4)
- added G***: LOGO, LOGO, F.Cu at (337.8, 108.8)
- added G***: LOGO, LOGO, B.Cu at (277.4, 126.7)
- added G***: LOGO, LOGO, B.Cu at (386.1, 128.7)
- added G***: LOGO, LOGO, B.Cu at (114.3, 100.0)
- moved G*** 3.14 mm to (366.0, 59.0)
Other:
- board text added: "Scan pwease:3"
- board text removed: "Don't, I warned you"
- board text removed: "THOCKS!"
- board text removed: "This One"
- board text removed: "This keyboard is cursed with functionality and coolness, use with caution:)"
